Commit message: controls working, now adding sensors

File: src/robot_description/urdf/macros.xacro (robot description, xacro)
@@ -19,6 +19,6 @@
                 />
     </macro>
-    <macro name="wheel" params="lr tY">
-      <link name="${lr}_wheel">
+    <macro name="wheel" params="lr fb tY tX">
+      <link name="${lr}_${fb}_wheel">
         <collision>
           <origin xyz="0 0 0" rpy="0 ${PI/2} ${PI/2}" />
@@ -40,5 +40,5 @@
         </inertial>
       </link>
-      <gazebo reference="${lr}_wheel">
+      <gazebo reference="${lr}_${fb}_wheel">
         <mu1 value="1.0"/>
         <mu2 value="1.0"/>
@@ -48,17 +48,21 @@
         <material>Gazebo/Black</material>
       </gazebo>
-      <joint name="${lr}_wheel_hinge" type="continuous">
+      <joint name="${lr}_${fb}_wheel_hinge" type="continuous">
         <parent link="chassis"/>
-        <child link="${lr}_wheel"/>
-      <origin xyz="${-wheelPos+chassisLength/2} ${tY*wheelWidth/2+tY*chassisWidth/2} ${wheelRadius}" rpy="0 0 0" />
+        <child link="${lr}_${fb}_wheel"/>
+        <origin xyz="${tX * (chassisLength - wheelPos) / 2}
+                     ${tY * wheelWidth / 2 + tY * chassisWidth / 2}
+                     ${wheelRadius}"
+                rpy="0 0 0" />
         <axis xyz="0 1 0" rpy="0 0 0" />
         <limit effort="100" velocity="100"/>
         <joint_properties damping="0.0" friction="0.0"/>
       </joint>
-      <transmission name="${lr}_trans">
+      <transmission name="${lr}_${fb}_trans">
         <type>transmission_interface/SimpleTransmission</type>
-        <joint name="${lr}_wheel_hinge"/>
-        <actuator name="${lr}Motor">
-          <hardwareInterface>EffortJointInterface</hardwareInterface>
+        <joint name="${lr}_${fb}_wheel_hinge">
+          <hardwareInterface>hardware_interface/EffortJointInterface</hardwareInterface>
+        </joint>
+        <actuator name="${lr}_${fb}_motor">
           <mechanicalReduction>10</mechanicalReduction>
         </actuator>

File: src/robot_description/urdf/robot.xacro (robot description, xacro)
@@ -6,18 +6,20 @@
     <xacro:property name="PI" value="3.1415926535897931"/>
   	<xacro:property name="chassisHeight" value="0.1"/>
-  	<xacro:property name="chassisLength" value="0.4"/>
-  	<xacro:property name="chassisWidth" value="0.2"/>
+  	<xacro:property name="chassisLength" value="1.2"/>
+  	<xacro:property name="chassisWidth" value="0.8"/>
   	<xacro:property name="chassisMass" value="50"/>
-  	<xacro:property name="casterRadius" value="0.05"/>
-  	<xacro:property name="casterMass" value="5"/>
-  	<xacro:property name="wheelWidth" value="0.05"/>
-  	<xacro:property name="wheelRadius" value="0.1"/>
+    <xacro:property name="towerHeight" value="1"/>
+    <xacro:property name="towerLength" value=".5"/>
+    <xacro:property name="towerWidth" value=".5"/>
+    <xacro:property name="towerMass" value="50"/>
+  	<xacro:property name="wheelWidth" value="0.1"/>
+  	<xacro:property name="wheelRadius" value="0.2"/>
   	<xacro:property name="wheelPos" value="0.2"/>
   	<xacro:property name="wheelMass" value="5"/>
   	<xacro:property name="cameraSize" value="0.05"/>
   	<xacro:property name="cameraMass" value="0.1"/>
-    <link name="footprint" />
+    <link name="base_link" />
     <joint name="base_joint" type="fixed">
-      <parent link="footprint"/>
+      <parent link="base_link"/>
       <child link="chassis"/>
     </joint>
@@ -34,5 +36,5 @@
            <box size="${chassisLength} ${chassisWidth} ${chassisHeight}"/>
   	     </geometry>
-  	       <material name="orange"/>
+  	       <material name="grey"/>
   	   </visual>
   	   <inertial>
@@ -41,30 +43,34 @@
   	     <box_inertia m="${chassisMass}" x="${chassisLength}" y="${chassisWidth}" z="${chassisHeight}"/>
   	   </inertial>
-  	</link>
-    <joint name="fixed" type="fixed">
-      <parent link="chassis"/>
-      <child link="caster_wheel"/>
+    </link>
+    <joint name = "tower" type = "fixed">
+      <parent link = "chassis"/>
+      <child link = "controlTower"/>
+      <origin xyz="0 0 ${wheelRadius + chassisHeight / 2}"/>
     </joint>
-    <link name="caster_wheel">
+    <!-- ${wheelRadius + (chassisHeight + towerHeight) / 2} -->
+    <link name = "controlTower">
       <collision>
-        <origin xyz="${casterRadius-chassisLength/2} 0 ${casterRadius-chassisHeight+wheelRadius}" rpy="0 0 0"/>
+        <origin xyz="0 0 ${towerHeight / 2}" rpy="0 0 0"/>
         <geometry>
-          <sphere radius="${casterRadius}"/>
+           <box size="${towerLength} ${towerWidth} ${towerHeight}"/>
         </geometry>
       </collision>
       <visual>
-        <origin xyz="${casterRadius-chassisLength/2} 0 ${casterRadius-chassisHeight+wheelRadius}" rpy="0 0 0"/>
+        <origin xyz="0 0 ${towerHeight / 2}" rpy="0 0 0"/>
         <geometry>
-          <sphere radius="${casterRadius}"/>
+           <box size="${towerLength} ${towerWidth} ${towerHeight}"/>
         </geometry>
-        <material name="red"/>
+        <material name="black"/>
       </visual>
       <inertial>
-        <origin xyz="${casterRadius-chassisLength/2} 0 ${casterRadius-chassisHeight+wheelRadius}" rpy="0 0 0"/>
-        <mass value="${casterMass}"/>
-        <sphere_inertia m="${casterMass}" r="${casterRadius}"/>
+        <origin xyz="0 0 ${wheelRadius + chassisHeight + towerHeight / 2}" rpy="0 0 0"/>
+        <mass value="${towerMass}"/>
+        <box_inertia m="${towerMass}" x="${towerLength}" y="${towerWidth}" z="${towerHeight}"/>
       </inertial>
-    </link>
-    <wheel lr="left" tY="1"/>
-    <wheel lr="right" tY="-1"/>
+   </link>
+   <xacro:wheel lr="left" fb="front" tY="1" tX = "1"/>
+   <xacro:wheel lr="right" fb="front" tY="-1" tX = "1"/>
+   <xacro:wheel lr="left" fb = "back" tY="1" tX = "-1"/>
+   <xacro:wheel lr="right" fb = "back" tY="-1" tX = "-1"/>
   </robot>

Commit message: adding rtabmap integration + localization

File: src/robot_description/urdf/macros.xacro (robot description, xacro)
@@ -53,5 +53,5 @@
         <origin xyz="${tX * (chassisLength - wheelPos) / 2}
                      ${tY * wheelWidth / 2 + tY * chassisWidth / 2}
-                     ${wheelRadius}"
+                     0"
                 rpy="0 0 0" />
         <axis xyz="0 1 0" rpy="0 0 0" />

File: src/robot_description/urdf/robot.xacro (robot description, xacro)
@@ -8,23 +8,24 @@
   	<xacro:property name="chassisLength" value="1.2"/>
   	<xacro:property name="chassisWidth" value="0.8"/>
-  	<xacro:property name="chassisMass" value="50"/>
+  	<xacro:property name="chassisMass" value="200"/>
     <xacro:property name="towerHeight" value="1"/>
     <xacro:property name="towerLength" value=".5"/>
     <xacro:property name="towerWidth" value=".5"/>
-    <xacro:property name="towerMass" value="50"/>
+    <xacro:property name="towerMass" value="100"/>
   	<xacro:property name="wheelWidth" value="0.1"/>
   	<xacro:property name="wheelRadius" value="0.2"/>
   	<xacro:property name="wheelPos" value="0.2"/>
-  	<xacro:property name="wheelMass" value="5"/>
+  	<xacro:property name="wheelMass" value="50"/>
   	<xacro:property name="cameraSize" value="0.05"/>
-  	<xacro:property name="cameraMass" value="0.1"/>
+  	<xacro:property name="cameraMass" value="5"/>
     <link name="base_link" />
     <joint name="base_joint" type="fixed">
       <parent link="base_link"/>
       <child link="chassis"/>
+      <origin xyz="0 0 ${wheelRadius}"/>
     </joint>
   	<link name='chassis'>
   	   <collision>
-  	     <origin xyz="0 0 ${wheelRadius}" rpy="0 0 0"/>
+  	     <origin xyz="0 0 0" rpy="0 0 0"/>
   	     <geometry>
   	        <box size="${chassisLength} ${chassisWidth} ${chassisHeight}"/>
@@ -32,5 +33,5 @@
   	   </collision>
        <visual>
-  	     <origin xyz="0 0 ${wheelRadius}" rpy="0 0 0"/>
+  	     <origin xyz="0 0 0" rpy="0 0 0"/>
   	     <geometry>
            <box size="${chassisLength} ${chassisWidth} ${chassisHeight}"/>
@@ -39,5 +40,5 @@
   	   </visual>
   	   <inertial>
-  	     <origin xyz="0 0 ${wheelRadius}" rpy="0 0 0"/>
+  	     <origin xyz="0 0 0" rpy="0 0 0"/>
   	     <mass value="${chassisMass}"/>
   	     <box_inertia m="${chassisMass}" x="${chassisLength}" y="${chassisWidth}" z="${chassisHeight}"/>
@@ -47,5 +48,5 @@
       <parent link = "chassis"/>
       <child link = "controlTower"/>
-      <origin xyz="0 0 ${wheelRadius + chassisHeight / 2}"/>
+      <origin xyz="0 0 ${chassisHeight / 2}"/>
     </joint>
     <!-- ${wheelRadius + (chassisHeight + towerHeight) / 2} -->
@@ -65,5 +66,5 @@
       </visual>
       <inertial>
-        <origin xyz="0 0 ${wheelRadius + chassisHeight + towerHeight / 2}" rpy="0 0 0"/>
+        <origin xyz="0 0 ${towerHeight / 2}" rpy="0 0 0"/>
         <mass value="${towerMass}"/>
         <box_inertia m="${towerMass}" x="${towerLength}" y="${towerWidth}" z="${towerHeight}"/>
@@ -76,16 +77,16 @@
    <joint name = "lidar" type = "fixed">
     <parent link = "controlTower"/>
-    <child link = "hokuyo_link"/>
-    <origin xyz="0 0 ${towerHeight}"/>
+    <child link = "lidar_link"/>
+    <origin xyz="${towerLength / 2} 0 ${towerHeight *3 / 4}"/>
   </joint>
-  <link name="hokuyo_link">
+  <link name="lidar_link">
     <collision>
-      <origin xyz="0 0 .05" rpy="0 0 0"/>
+      <origin xyz="${cameraSize / 2} 0 ${cameraSize / 2}" rpy="0 0 0"/>
       <geometry>
-        <box size="0.1 0.1 0.1"/>
+        <box size="${cameraSize / 2} ${cameraSize / 2} ${cameraSize / 2}"/>
       </geometry>
     </collision>
     <visual>
-      <origin xyz="0 0 .05" rpy="0 0 0"/>
+      <origin xyz= "${cameraSize / 2} 0 ${cameraSize / 2}" />
       <geometry>
         <!-- <mesh filename="package://rrbot_description/meshes/hokuyo.dae"/> -->
@@ -94,8 +95,35 @@
     </visual>
     <inertial>
-      <mass value="1e-5" />
-      <origin xyz="0 0 0" rpy="0 0 0"/>
-      <inertia ixx="1e-6" ixy="0" ixz="0" iyy="1e-6" iyz="0" izz="1e-6" />
+      <mass value="${cameraMass}" />
+      <origin xyz="${cameraSize / 2} 0 ${cameraSize / 2}" rpy="0 0 0"/>
+      <xacro:box_inertia m = "${cameraMass}" x = "${cameraSize}"
+                         y = "${cameraSize}" z = "${cameraSize}"/>
     </inertial>
   </link>
+  <joint name = "camera" type = "fixed">
+   <parent link = "controlTower"/>
+   <child link = "camera_link"/>
+   <origin xyz="${towerLength / 2} 0 ${towerHeight / 2}"/>
+ </joint>
+   <link name="camera_link">
+     <collision>
+       <origin xyz="${cameraSize / 2} 0 ${cameraSize / 2}" rpy="0 0 0"/>
+       <geometry>
+         <box size="${cameraSize / 2} ${cameraSize / 2} ${cameraSize / 2}"/>
+       </geometry>
+     </collision>
+     <visual>
+       <origin xyz= "${cameraSize / 2} 0 ${cameraSize / 2}" />
+       <geometry>
+         <!-- <mesh filename="package://rrbot_description/meshes/hokuyo.dae"/> -->
+         <box size="0.1 0.1 0.1"/>
+       </geometry>
+     </visual>
+     <inertial>
+       <mass value="${cameraMass}" />
+       <origin xyz="${cameraSize / 2} 0 ${cameraSize / 2}" rpy="0 0 0"/>
+       <xacro:box_inertia m = "${cameraMass}" x = "${cameraSize}"
+                          y = "${cameraSize}" z = "${cameraSize}"/>
+     </inertial>
+   </link>
 </robot>
