Commit message: added sensors

File: src/robot_description/urdf/robot.xacro (robot description, xacro)
@@ -74,3 +74,28 @@
    <xacro:wheel lr="left" fb = "back" tY="1" tX = "-1"/>
    <xacro:wheel lr="right" fb = "back" tY="-1" tX = "-1"/>
-  </robot>
+   <joint name = "lidar" type = "fixed">
+    <parent link = "controlTower"/>
+    <child link = "hokuyo_link"/>
+    <origin xyz="0 0 ${towerHeight}"/>
+  </joint>
+  <link name="hokuyo_link">
+    <collision>
+      <origin xyz="0 0 .05" rpy="0 0 0"/>
+      <geometry>
+        <box size="0.1 0.1 0.1"/>
+      </geometry>
+    </collision>
+    <visual>
+      <origin xyz="0 0 .05" rpy="0 0 0"/>
+      <geometry>
+        <!-- <mesh filename="package://rrbot_description/meshes/hokuyo.dae"/> -->
+        <box size="0.1 0.1 0.1"/>
+      </geometry>
+    </visual>
+    <inertial>
+      <mass value="1e-5" />
+      <origin xyz="0 0 0" rpy="0 0 0"/>
+      <inertia ixx="1e-6" ixy="0" ixz="0" iyy="1e-6" iyz="0" izz="1e-6" />
+    </inertial>
+  </link>
+</robot>

Commit message: rtabmap works, added slam package

File: src/robot_description/urdf/robot.xacro (robot description, xacro)
@@ -17,5 +17,5 @@
   	<xacro:property name="wheelPos" value="0.2"/>
   	<xacro:property name="wheelMass" value="50"/>
-  	<xacro:property name="cameraSize" value="0.05"/>
+  	<xacro:property name="cameraSize" value="0.1"/>
   	<xacro:property name="cameraMass" value="5"/>
     <link name="base_link" />
@@ -75,55 +75,56 @@
    <xacro:wheel lr="left" fb = "back" tY="1" tX = "-1"/>
    <xacro:wheel lr="right" fb = "back" tY="-1" tX = "-1"/>
-   <joint name = "lidar" type = "fixed">
+   <joint name = "camera" type = "fixed">
     <parent link = "controlTower"/>
-    <child link = "lidar_link"/>
-    <origin xyz="${towerLength / 2} 0 ${towerHeight *3 / 4}"/>
+    <child link = "camera_link"/>
+    <origin xyz="${towerLength / 2 + cameraSize / 2} 0 ${towerHeight * 3 / 4}"
+             />
   </joint>
-  <link name="lidar_link">
+  <link name="camera_link">
     <collision>
-      <origin xyz="${cameraSize / 2} 0 ${cameraSize / 2}" rpy="0 0 0"/>
+      <origin xyz="0 0 0" rpy="0 0 0"/>
       <geometry>
-        <box size="${cameraSize / 2} ${cameraSize / 2} ${cameraSize / 2}"/>
+        <box size="${cameraSize} ${cameraSize} ${cameraSize}"/>
       </geometry>
     </collision>
     <visual>
-      <origin xyz= "${cameraSize / 2} 0 ${cameraSize / 2}" />
+      <origin xyz= "0 0 0" />
       <geometry>
         <!-- <mesh filename="package://rrbot_description/meshes/hokuyo.dae"/> -->
-        <box size="0.1 0.1 0.1"/>
+        <box size="${cameraSize} ${cameraSize} ${cameraSize}"/>
       </geometry>
     </visual>
     <inertial>
       <mass value="${cameraMass}" />
-      <origin xyz="${cameraSize / 2} 0 ${cameraSize / 2}" rpy="0 0 0"/>
+      <origin xyz="0 0 0" rpy="0 0 0"/>
       <xacro:box_inertia m = "${cameraMass}" x = "${cameraSize}"
                          y = "${cameraSize}" z = "${cameraSize}"/>
     </inertial>
   </link>
-  <joint name = "camera" type = "fixed">
+  <joint name = "lidar" type = "fixed">
    <parent link = "controlTower"/>
-   <child link = "camera_link"/>
-   <origin xyz="${towerLength / 2} 0 ${towerHeight / 2}"/>
- </joint>
-   <link name="camera_link">
-     <collision>
-       <origin xyz="${cameraSize / 2} 0 ${cameraSize / 2}" rpy="0 0 0"/>
-       <geometry>
-         <box size="${cameraSize / 2} ${cameraSize / 2} ${cameraSize / 2}"/>
-       </geometry>
-     </collision>
-     <visual>
-       <origin xyz= "${cameraSize / 2} 0 ${cameraSize / 2}" />
-       <geometry>
-         <!-- <mesh filename="package://rrbot_description/meshes/hokuyo.dae"/> -->
-         <box size="0.1 0.1 0.1"/>
-       </geometry>
-     </visual>
-     <inertial>
-       <mass value="${cameraMass}" />
-       <origin xyz="${cameraSize / 2} 0 ${cameraSize / 2}" rpy="0 0 0"/>
-       <xacro:box_inertia m = "${cameraMass}" x = "${cameraSize}"
-                          y = "${cameraSize}" z = "${cameraSize}"/>
-     </inertial>
-   </link>
+   <child link = "lidar_link"/>
+   <origin xyz="${towerLength / 2 + cameraSize / 2} 0 ${towerHeight / 4}"/>
+  </joint>
+  <link name="lidar_link">
+   <collision>
+     <origin xyz="0 0 0" rpy="0 0 0"/>
+     <geometry>
+       <box size="${cameraSize} ${cameraSize} ${cameraSize}"/>
+     </geometry>
+   </collision>
+   <visual>
+     <origin xyz= "0 0 0" />
+     <geometry>
+       <!-- <mesh filename="package://rrbot_description/meshes/hokuyo.dae"/> -->
+       <box size="${cameraSize} ${cameraSize} ${cameraSize}"/>
+     </geometry>
+   </visual>
+   <inertial>
+     <mass value="${cameraMass}" />
+     <origin xyz="0 0 0" rpy="0 0 0"/>
+     <xacro:box_inertia m = "${cameraMass}" x = "${cameraSize}"
+                        y = "${cameraSize}" z = "${cameraSize}"/>
+   </inertial>
+ </link>
 </robot>

Commit message: working rtabmap

File: src/robot_description/urdf/robot.xacro (robot description, xacro)
@@ -76,55 +76,61 @@
    <xacro:wheel lr="right" fb = "back" tY="-1" tX = "-1"/>
    <joint name = "camera" type = "fixed">
-    <parent link = "controlTower"/>
-    <child link = "camera_link"/>
-    <origin xyz="${towerLength / 2 + cameraSize / 2} 0 ${towerHeight * 3 / 4}"
-             />
-  </joint>
-  <link name="camera_link">
-    <collision>
-      <origin xyz="0 0 0" rpy="0 0 0"/>
-      <geometry>
-        <box size="${cameraSize} ${cameraSize} ${cameraSize}"/>
-      </geometry>
-    </collision>
-    <visual>
-      <origin xyz= "0 0 0" />
-      <geometry>
-        <!-- <mesh filename="package://rrbot_description/meshes/hokuyo.dae"/> -->
-        <box size="${cameraSize} ${cameraSize} ${cameraSize}"/>
-      </geometry>
-    </visual>
-    <inertial>
-      <mass value="${cameraMass}" />
-      <origin xyz="0 0 0" rpy="0 0 0"/>
-      <xacro:box_inertia m = "${cameraMass}" x = "${cameraSize}"
-                         y = "${cameraSize}" z = "${cameraSize}"/>
-    </inertial>
-  </link>
-  <joint name = "lidar" type = "fixed">
-   <parent link = "controlTower"/>
-   <child link = "lidar_link"/>
-   <origin xyz="${towerLength / 2 + cameraSize / 2} 0 ${towerHeight / 4}"/>
-  </joint>
-  <link name="lidar_link">
-   <collision>
-     <origin xyz="0 0 0" rpy="0 0 0"/>
-     <geometry>
-       <box size="${cameraSize} ${cameraSize} ${cameraSize}"/>
-     </geometry>
-   </collision>
-   <visual>
-     <origin xyz= "0 0 0" />
-     <geometry>
-       <!-- <mesh filename="package://rrbot_description/meshes/hokuyo.dae"/> -->
-       <box size="${cameraSize} ${cameraSize} ${cameraSize}"/>
-     </geometry>
-   </visual>
-   <inertial>
-     <mass value="${cameraMass}" />
-     <origin xyz="0 0 0" rpy="0 0 0"/>
-     <xacro:box_inertia m = "${cameraMass}" x = "${cameraSize}"
-                        y = "${cameraSize}" z = "${cameraSize}"/>
-   </inertial>
- </link>
+     <parent link = "controlTower"/>
+     <child link = "camera_link"/>
+     <origin xyz="${towerLength / 2 + cameraSize / 2} 0 ${towerHeight * 3 / 4}"/>
+   </joint>
+   <link name="camera_link">
+     <collision>
+       <origin xyz="0 0 0" rpy="0 0 0"/>
+       <geometry>
+         <box size="${cameraSize} ${cameraSize} ${cameraSize}"/>
+       </geometry>
+     </collision>
+     <visual>
+       <origin xyz= "0 0 0" />
+       <geometry>
+         <!-- <mesh filename="package://rrbot_description/meshes/hokuyo.dae"/> -->
+         <box size="${cameraSize} ${cameraSize} ${cameraSize}"/>
+       </geometry>
+     </visual>
+     <inertial>
+       <mass value="${cameraMass}" />
+       <origin xyz="0 0 0" rpy="0 0 0"/>
+       <xacro:box_inertia m = "${cameraMass}" x = "${cameraSize}"
+         y = "${cameraSize}" z = "${cameraSize}"/>
+     </inertial>
+   </link>
+   <joint name="camera_optical_joint" type="fixed">
+   <origin xyz="0 0 0" rpy="${PI/2} ${PI} ${PI/2}"/>
+   <parent link="camera_link"/>
+   <child link="camera_link_optical"/>
+   </joint>
+   <link name="camera_link_optical">
+   </link>
+   <joint name = "lidar" type = "fixed">
+       <parent link = "controlTower"/>
+       <child link = "lidar_link"/>
+       <origin xyz="${towerLength / 2 + cameraSize / 2} 0 ${towerHeight / 4}"/>
+   </joint>
+   <link name="lidar_link">
+     <collision>
+       <origin xyz="0 0 0" rpy="0 0 0"/>
+       <geometry>
+         <box size="${cameraSize} ${cameraSize} ${cameraSize}"/>
+       </geometry>
+     </collision>
+     <visual>
+       <origin xyz= "0 0 0" />
+       <geometry>
+         <!-- <mesh filename="package://rrbot_description/meshes/hokuyo.dae"/> -->
+         <box size="${cameraSize} ${cameraSize} ${cameraSize}"/>
+       </geometry>
+     </visual>
+     <inertial>
+       <mass value="${cameraMass}" />
+       <origin xyz="0 0 0" rpy="0 0 0"/>
+       <xacro:box_inertia m = "${cameraMass}" x = "${cameraSize}"
+         y = "${cameraSize}" z = "${cameraSize}"/>
+     </inertial>
+   </link>
 </robot>

Commit message: localization needs tuning

File: src/robot_description/urdf/robot.xacro (robot description, xacro)
@@ -6,14 +6,14 @@
     <xacro:property name="PI" value="3.1415926535897931"/>
   	<xacro:property name="chassisHeight" value="0.1"/>
-  	<xacro:property name="chassisLength" value="1.2"/>
-  	<xacro:property name="chassisWidth" value="0.8"/>
+  	<xacro:property name="chassisLength" value=".6"/>
+  	<xacro:property name="chassisWidth" value="0.4"/>
   	<xacro:property name="chassisMass" value="200"/>
     <xacro:property name="towerHeight" value="1"/>
-    <xacro:property name="towerLength" value=".5"/>
-    <xacro:property name="towerWidth" value=".5"/>
+    <xacro:property name="towerLength" value=".3"/>
+    <xacro:property name="towerWidth" value=".3"/>
     <xacro:property name="towerMass" value="100"/>
-  	<xacro:property name="wheelWidth" value="0.1"/>
-  	<xacro:property name="wheelRadius" value="0.2"/>
-  	<xacro:property name="wheelPos" value="0.2"/>
+  	<xacro:property name="wheelWidth" value="0.05"/>
+  	<xacro:property name="wheelRadius" value="0.1"/>
+  	<xacro:property name="wheelPos" value="0.1"/>
   	<xacro:property name="wheelMass" value="50"/>
   	<xacro:property name="cameraSize" value="0.1"/>
@@ -107,4 +107,10 @@
    </joint>
    <link name="camera_link_optical">
+     <collision>
+       <origin xyz="0 0 0" rpy="0 0 0"/>
+       <geometry>
+         <box size="${cameraSize} ${cameraSize} ${cameraSize}"/>
+       </geometry>
+     </collision>
    </link>
    <joint name = "lidar" type = "fixed">

Commit message: architecture for slam done, need to tune

File: src/robot_description/urdf/robot.xacro (robot description, xacro)
@@ -6,5 +6,5 @@
     <xacro:property name="PI" value="3.1415926535897931"/>
   	<xacro:property name="chassisHeight" value="0.1"/>
-  	<xacro:property name="chassisLength" value=".6"/>
+  	<xacro:property name="chassisLength" value=".4"/>
   	<xacro:property name="chassisWidth" value="0.4"/>
   	<xacro:property name="chassisMass" value="200"/>
